File: Walkman-in-2026/Walkman-in-2026.kicad_pcb (KiCad board)
At the start: 2 copper layers, 1 part

Commit message: moving on to the pcb editor
Parts:
- removed REF**: XIAO-ESP32-S3-DIP, More XIAO:XIAO-ESP32-S3-DIP
- added C1: 2.2, Capacitor_THT:C_Disc_D3.0mm_W1.6mm_P2.50mm, F.Cu at (123.0, 111.0)
- added C10: 10, Capacitor_THT:C_Radial_D5.0mm_H5.0mm_P2.00mm, F.Cu at (118.5, 111.5)
- added C2: 2.2, Capacitor_THT:C_Disc_D3.0mm_W1.6mm_P2.50mm, F.Cu at (123.0, 114.2)
- added C3: 2.2, Capacitor_THT:C_Radial_D5.0mm_H5.0mm_P2.00mm, F.Cu at (110.0, 98.0)
- added C5: 2.2, Capacitor_THT:C_Radial_D5.0mm_H5.0mm_P2.00mm, F.Cu at (110.0, 104.5)
- added C6: 0.1, Capacitor_THT:C_Disc_D3.0mm_W1.6mm_P2.50mm, F.Cu at (123.0, 117.3)
- added C7: 0.1, Capacitor_THT:C_Disc_D3.0mm_W1.6mm_P2.50mm, F.Cu at (123.0, 120.5)
- added C8: 0.1, Capacitor_THT:C_Disc_D3.0mm_W1.6mm_P2.50mm, F.Cu at (123.0, 123.7)
- added C9: 0.1, Capacitor_THT:C_Radial_D5.0mm_H5.0mm_P2.00mm, F.Cu at (112.0, 111.5)
- added J1: AudioJack3, Connector_Audio:Jack_3.5mm_CUI_SJ1-3513N_Horizontal, F.Cu at (94.5, 102.0)
- added J2: Micro_SD_Card, Connector_Card:microSD_HC_Molex_47219-2001, F.Cu at (135.5, 117.5)
- added Q1: BSS138, Package_TO_SOT_SMD:SOT-23, F.Cu at (130.5, 99.5)
- added Q2: BSS138, Package_TO_SOT_SMD:SOT-23, F.Cu at (130.5, 104.0)
- added R1: 33, Resistor_THT:R_Axial_DIN0207_L6.3mm_D2.5mm_P7.62mm_Horizontal, F.Cu at (78.7, 116.0)
- added R10: 10k, Resistor_THT:R_Axial_DIN0207_L6.3mm_D2.5mm_P7.62mm_Horizontal, F.Cu at (78.8, 87.7)
- added R11: 10k, Resistor_THT:R_Axial_DIN0207_L6.3mm_D2.5mm_P7.62mm_Horizontal, F.Cu at (78.8, 77.0)
- added R12: 470, Resistor_THT:R_Axial_DIN0207_L6.3mm_D2.5mm_P7.62mm_Horizontal, F.Cu at (83.0, 108.2)
- added R13: 470, Resistor_THT:R_Axial_DIN0207_L6.3mm_D2.5mm_P7.62mm_Horizontal, F.Cu at (86.5, 108.3)
- added R2: 1k, Resistor_THT:R_Axial_DIN0207_L6.3mm_D2.5mm_P7.62mm_Horizontal, F.Cu at (88.7, 116.0)
- added R3: 1k, Resistor_THT:R_Axial_DIN0207_L6.3mm_D2.5mm_P7.62mm_Horizontal, F.Cu at (98.7, 116.0)
- added R4: 1k, Resistor_THT:R_Axial_DIN0207_L6.3mm_D2.5mm_P7.62mm_Horizontal, F.Cu at (108.7, 116.0)
- added R5: 1k, Resistor_THT:R_Axial_DIN0207_L6.3mm_D2.5mm_P7.62mm_Horizontal, F.Cu at (78.7, 111.5)
- added R6: 1k, Resistor_THT:R_Axial_DIN0207_L6.3mm_D2.5mm_P7.62mm_Horizontal, F.Cu at (88.7, 111.5)
- added R7: 10k, Resistor_THT:R_Axial_DIN0207_L6.3mm_D2.5mm_P7.62mm_Horizontal, F.Cu at (98.7, 111.5)
- added R8: 10k, Resistor_THT:R_Axial_DIN0207_L6.3mm_D2.5mm_P7.62mm_Horizontal, F.Cu at (79.0, 108.0)
- added R9: 10k, Resistor_THT:R_Axial_DIN0207_L6.3mm_D2.5mm_P7.62mm_Horizontal, F.Cu at (78.8, 98.0)
- added SW1: SW_Push, Button_Switch_THT:SW_PUSH_6mm, F.Cu at (79.3, 127.0)
- added SW2: SW_Push, Button_Switch_THT:SW_PUSH_6mm, F.Cu at (87.8, 127.0)
- added SW3: SW_Push, Button_Switch_THT:SW_PUSH_6mm, F.Cu at (96.4, 127.0)
- added SW4: SW_SPST, Button_Switch_THT:SW_SPST_Omron_B3F-315x_Angled, F.Cu at (166.0, 98.5)
- added SW5: SW_Push, Button_Switch_THT:SW_PUSH_6mm, F.Cu at (105.0, 127.0)
- added SW6: SW_Push, Button_Switch_THT:SW_PUSH_6mm, F.Cu at (113.5, 127.0)
- added U1: XIAO-ESP32-S3-DIP, More_XIAO_Series_Footprints:XIAO-ESP32-S3-DIP, F.Cu at (155.5, 117.2)
- added U2: HS1602A-B, EasyEDALibrary:LCD1602, F.Cu at (124.0, 76.0)
- added U3: PCM5102, Package_SO:TSSOP-20_4.4x6.5mm_P0.65mm, F.Cu at (118.0, 101.5)
- added U4: PCF8574P, Package_DIP:DIP-16_W7.62mm, F.Cu at (136.3, 104.5)

Commit message: May 3rd (end of worlds)
Parts:
- moved R5 165.3 mm to (243.0, 93.8), turned to 90 degrees
- moved R6 158.8 mm to (246.5, 93.6), turned to 90 degrees
- moved SW2 145.3 mm to (226.3, 83.0)
- moved SW1 145.3 mm to (217.8, 83.0)
- moved SW3 145.3 mm to (234.8, 83.0)
- moved SW5 145.3 mm to (243.4, 83.0)
- moved SW6 145.3 mm to (251.9, 83.0)
- moved R2 144.1 mm to (231.0, 93.6), turned to 90 degrees
- moved R13 139.6 mm to (225.5, 95.3)
- moved R3 138.1 mm to (235.0, 93.8), turned to 90 degrees
- moved R12 137.1 mm to (219.5, 95.5)
- moved R4 132.2 mm to (239.0, 93.6), turned to 90 degrees
- moved J1 116.1 mm to (208.5, 79.7), turned to -90 degrees
- moved U2 104.9 mm to (220.6, 117.0)
- moved R11 98.5 mm to (170.7, 112.5), turned to 0 degrees
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Routing:
- net GND: track 0.00 -> 293.5 mm, vias 0 -> 5
- net +3.3V: track 0.00 -> 139.9 mm, vias 0 -> 3
- net +5V: track 0.00 -> 118.7 mm, vias 0 -> 1
- net +3V3: track 0.00 -> 102.8 mm, vias 0 -> 1
- net Net-(U1-GPIO1_A0_D0): track 0.00 -> 74.2 mm
- net Net-(J2-DAT3/CD): track 0.00 -> 61.7 mm
- net Net-(U2-DB5): track 0.00 -> 57.5 mm
- net Net-(U2-DB7): track 0.00 -> 56.5 mm
- net Net-(U3-OUTR): track 0.00 -> 55.2 mm, vias 0 -> 1
- net Net-(U2-DB6): track 0.00 -> 53.4 mm
- net Net-(U2-LED+): track 0.00 -> 50.4 mm
- net Net-(U3-OUTL): track 0.00 -> 50.4 mm, vias 0 -> 1
- net Net-(Q1-G): track 0.00 -> 49.9 mm, vias 0 -> 1
- net Net-(U2-DB4): track 0.00 -> 48.8 mm
- net Net-(J2-DAT0): track 0.00 -> 47.4 mm
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
Commit message: may 6 session
Parts:
- moved Q1 2.55 mm to (167.0, 110.5)
- moved R10 1.00 mm to (168.0, 128.0)
- moved U1 0.42 mm to (173.4, 85.5)
Routing:
- net Net-(U1-GPIO1_A0_D0): track 74.2 -> 176.7 mm
- net Net-(SW4-A): track 0.00 -> 91.3 mm
- net Net-(R5-Pad1): track 0.00 -> 27.0 mm
- net Net-(R4-Pad1): track 0.00 -> 21.8 mm
- net Net-(R2-Pad1): track 0.00 -> 21.2 mm
- net Net-(R3-Pad1): track 0.00 -> 19.1 mm
- net +3V3: track 102.8 -> 120.4 mm
- net Net-(C2-Pad2): track 14.5 -> 29.5 mm
- net GND: track 293.5 -> 300.8 mm
- net +5V: track 118.7 -> 112.7 mm
- net +3.3V: track 139.9 -> 142.7 mm
- net Net-(Q1-D): track 34.7 -> 36.7 mm
- net Net-(Q2-D): track 32.8 -> 31.4 mm
- net Net-(U1-GPIO3_A2_D2): track 32.3 -> 33.0 mm
- net Net-(J2-CLK): track 39.2 -> 39.9 mm
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Other:
- board outline added: 100 x 63.5 mm
